Commit message: feat: add MTC approach planning and MuJoCo replay
Build and audit the complete MoveIt model, raise the fuel opening with grounded body geometry, refresh reproducibility reports, and record the adopted RGB-D technical route.

File: assets/objects/fuel_tank/urdf/fuel_tank.urdf (robot description, URDF)
Before this commit: robot fuel_tank, 5 links, 4 joints
Links:
- added link tank_body_center
- link fuel_tank_body: geometry collision box size=0.8 0.19999999999999996 0.4; collision mesh filename=../meshes/body_00.stl
Joints:
- added joint tank_body_center_fixed: type fixed, parent fuel_tank_body, child tank_body_center, origin xyz=0 -0.099999999999999978 0.2 rpy=0 0 0
- joint fuel_tank_fixed: origin xyz=0 0.2 0.4 rpy=1.570796326794897 0 0 -> xyz=0 0.2 0.6 rpy=1.570796326794897 0 0
