Commit message: feat: checkpoint SDK readout, point clouds and pregrasp inputs
Integrate fixed-grasp target preparation, RGB-D reconstruction, voxel and
binary PCD inspection tools, with standalone point-cloud viewers and evidence.
Add AUBO SDK 0.23.1 read-only probes, RPC/RTDE captures and model comparisons.
Record confirmed camera-frame millimetres and flange_from_camera extrinsics.
Document the remaining MoveIt state and whole-trajectory execution work.
Keep vendor SDK binaries local; retain download instructions and file hashes.

Validation: SDK Release build, offline initialization and 26 API symbols pass.
Model provenance, calibration numerics and capture manifests pass; current E2
baseline and mixed trajectory replays pass. Scoped pytest: 125 passed,
17 failed and 31 setup errors, all from archived planning fixtures rejected
for stale scene hashes. Preserve those records and document fixture migration.

File: assets/objects/fuel_cap/urdf/fuel_cap.urdf (robot description, URDF)
Before this commit: robot fuel_cap_inspection, 5 links, 4 joints
Joints:
- joint cap_bottom_center_joint: origin xyz=0 0 -0.020 rpy=0 0 0 -> xyz=0 0 -0.020 rpy=0 0 1.5707963267948966
- joint cap_grip_center_joint: origin xyz=0 0 0.030 rpy=0 0 0 -> xyz=0 0 0.030 rpy=0 0 1.5707963267948966
- joint cap_grip_top_center_joint: origin xyz=0 0 0.0385 rpy=0 0 0 -> xyz=0 0 0.0385 rpy=0 0 1.5707963267948966
